Commit message: modified right_softhand_v3.urdf and generate new right_softhand_v3.xml

File: softhands_description/urdf/right_softhand_v3.urdf (robot description, URDF)
Before this commit: robot softhand, 35 links, 34 joints
Links:
- link right_hand_v3_index_distal_link: mass 0.0024034657 -> 0.009
- link right_hand_v3_index_distal_virtual_link: mass 0.0024034657 -> 0.009
- link right_hand_v3_little_distal_link: mass 0.0024034657 -> 0.009
- link right_hand_v3_little_distal_virtual_link: mass 0.0024034657 -> 0.009
- link right_hand_v3_middle_distal_link: mass 0.0024034657 -> 0.009
- link right_hand_v3_middle_distal_virtual_link: mass 0.0024034657 -> 0.009
- link right_hand_v3_ring_distal_link: mass 0.0024034657 -> 0.009
- link right_hand_v3_ring_distal_virtual_link: mass 0.0024034657 -> 0.009
- link right_hand_v3_thumb_distal_link: mass 0.0024034657 -> 0.009
- link right_hand_v3_thumb_distal_virtual_link: mass 0.0024034657 -> 0.009
Joints:
- joint right_hand_v3_index_distal_joint: origin xyz=10e-03 -0.000348650e-03 0.5e-03 rpy=0 0 0 -> xyz=9e-03 -0.000348650e-03 0.5e-03 rpy=0 0 0
- joint right_hand_v3_index_middle_joint: origin xyz=10e-03 0 0 rpy=0 0 0 -> xyz=9e-03 0 0 rpy=0 0 0
- joint right_hand_v3_index_proximal_joint: origin xyz=10e-03 0 0 rpy=0 0 0 -> xyz=9e-03 0 0 rpy=0 0 0
- joint right_hand_v3_little_distal_joint: origin xyz=10e-03 -0.000348650e-03 0.5e-03 rpy=0 0 0 -> xyz=9e-03 -0.000348650e-03 0.5e-03 rpy=0 0 0
- joint right_hand_v3_little_middle_joint: origin xyz=10e-03 0 0 rpy=0 0 0 -> xyz=9e-03 0 0 rpy=0 0 0
- joint right_hand_v3_little_proximal_joint: origin xyz=10e-03 0 0 rpy=0 0 0 -> xyz=9e-03 0 0 rpy=0 0 0
- joint right_hand_v3_middle_distal_joint: origin xyz=10e-03 -0.000348650e-03 0.5e-03 rpy=0 0 0 -> xyz=9e-03 -0.000348650e-03 0.5e-03 rpy=0 0 0
- joint right_hand_v3_middle_middle_joint: origin xyz=10e-03 0 0 rpy=0 0 0 -> xyz=9e-03 0 0 rpy=0 0 0
- joint right_hand_v3_middle_proximal_joint: origin xyz=10e-03 0 0 rpy=0 0 0 -> xyz=9e-03 0 0 rpy=0 0 0
- joint right_hand_v3_ring_distal_joint: origin xyz=10e-03 -0.000348650e-03 0.5e-03 rpy=0 0 0 -> xyz=9e-03 -0.000348650e-03 0.5e-03 rpy=0 0 0
- joint right_hand_v3_ring_middle_joint: origin xyz=10e-03 0 0 rpy=0 0 0 -> xyz=9e-03 0 0 rpy=0 0 0
- joint right_hand_v3_ring_proximal_joint: origin xyz=10e-03 0 0 rpy=0 0 0 -> xyz=9e-03 0 0 rpy=0 0 0
- joint right_hand_v3_thumb_distal_joint: origin xyz=10e-03 0 0 rpy=0 0 0 -> xyz=9e-03 0 0 rpy=0 0 0
- joint right_hand_v3_thumb_proximal_joint: origin xyz=10e-03 0 0 rpy=0 0 0 -> xyz=9e-03 0 0 rpy=0 0 0
